File: OpenKickstartSwitcher.kicad_pcb (KiCad board)
At the start: 2 copper layers, 25.7 x 79.2 mm, 13 parts, among them J1 Conn_01x03, J2 Conn_01x04, J4 Conn_01x03, J98 LOGO, J99 OSHW_LOGO, U1 KS_SOCKET, U2 M27C800, U3 7400

Commit message: Almost there...
Routing:
- net /a5: track 18.3 -> 19.1 mm
- net /a2: track 20.0 -> 20.6 mm
- net /a17: track 67.5 -> 67.0 mm
- net GND: vias 45 -> 57
Other:
- rule solder_mask_min_width: 0.25 -> 0.2
- board text added: "A19"

Commit message: Almost there... (again)
Routing:
- net GND: track 0.00 -> 2.26 mm
Changed lines of the file:
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@@
   (general
     (thickness 1.6)
-    (drawings 47)
-    (tracks 368)
+    (drawings 46)
+    (tracks 370)
     (zones 0)
     (modules 13)
@@
   (title_block
     (title OpenKickstartSwitcher)
-    (date 2018-04-21)
-    (rev V2)
+    (date 2018-12-22)
+    (rev V1cdtv)
     (company SukkoPera)
     (comment 1 "Inspired from work by Henryk Richter")
@@
     (39 F.Mask user)
     (44 Edge.Cuts user)
-    (49 F.Fab user hide)
+    (49 F.Fab user)
   )
   (setup
@@
     (mod_text_width 0.15)
     (pad_size 1.6 1.6)
-    (pad_drill 0.8)
+    (pad_drill 1)
     (pad_to_mask_clearance 0)
     (solder_mask_min_width 0.2)
@@
       (padsonsilk false)
       (subtractmaskfromsilk false)
-      (outputformat 4)
+      (outputformat 1)
       (mirror false)
       (drillshape 0)
@@
     (effects (font (size 0.8 0.7) (thickness 0.15)) (justify mirror))
   )
-  (gr_text "Licensed under\nCERN OHL v.1.2" (at 156.337 115.443 90) (layer B.SilkS)
+  (gr_text "Licensed under\nCERN OHL v.1.2" (at 156.972 115.824 90) (layer B.SilkS)
     (effects (font (size 1 1) (thickness 0.15)) (justify mirror))
   )
@@
     (arrow2b (pts (xy 152.019 171.45) (xy 150.892496 172.036421)))
   )
-  (gr_text "github.com/SukkoPera/\nOpenKickstartSwitcher" (at 161.671 115.316 90) (layer B.SilkS)
+  (gr_text "github.com/SukkoPera/\nOpenKickstartSwitcher" (at 161.036 116.078 90) (layer B.SilkS)
     (effects (font (size 1 1) (thickness 0.15)) (justify mirror))
   )
@@
     (effects (font (size 0.8 0.7) (thickness 0.15)))
   )
-  (target plus (at 169.291 165.1) (size 5) (width 0.15) (layer Edge.Cuts))
   (gr_arc (start 144.907 150.495) (end 144.907 151.765) (angle 90) (layer Edge.Cuts) (width 0.15))
   (gr_arc (start 150.749 153.035) (end 150.749 151.765) (angle 90) (layer Edge.Cuts) (width 0.15))
@@
   (via (at 167.386 152.527) (size 0.8) (drill 0.6) (layers F.Cu B.Cu) (net 5))
   (via (at 164.211 144.0688) (size 0.7) (drill 0.6) (layers F.Cu B.Cu) (net 5))
+  (segment (start 146.685 101.854) (end 146.685 102.98537) (width 0.4) (layer F.Cu) (net 5))
+  (segment (start 146.685 101.854) (end 146.685 100.72263) (width 0.4) (layer F.Cu) (net 5))
   (segment (start 148.844 89.281) (end 150.749 89.281) (width 0.4) (layer F.Cu) (net 6))
   (segment (start 146.304 134.911) (end 146.304 136.311) (width 0.4) (layer B.Cu) (net 6))
@@
     (connect_pads (clearance 0.1))
     (min_thickness 0.0254)
-    (fill yes (arc_segments 16) (thermal_gap 0.3) (thermal_bridge_width 0.5))
+    (fill yes (arc_segments 16) (thermal_gap 0.2) (thermal_bridge_width 0.5))
     (polygon
       (pts
@@
     (connect_pads (clearance 0.1))
     (min_thickness 0.0254)
-    (fill yes (arc_segments 16) (thermal_gap 0.3) (thermal_bridge_width 0.5))
+    (fill yes (arc_segments 16) (thermal_gap 0.2) (thermal_bridge_width 0.5))
     (polygon
       (pts

Commit message: Ready for V1-cdtv!
Parts:
- moved C1 0.38 mm to (146.7, 89.7)
- moved U3 0.38 mm to (152.0, 96.0)
Routing:
- net VCC: track 142.6 -> 140.9 mm
- net /sw17: track 25.6 -> 24.1 mm
- net Net-(U2-Pad2): track 60.2 -> 60.7 mm
Other:
- board size 25.7 x 79.2 mm -> 25.7 x 78.5 mm
